Commit message: Pi stuff

File: description/lidar.xacro (robot description, xacro)
@@ -2,9 +2,9 @@
 <robot xmlns:xacro="http://www.ros.org/wiki/xacro" >
     <joint name="laser_joint" type="fixed">
-        <parent link="chassis"/>
-        <child link="laser_frame"/>
+        <parent link="base_link"/>
+        <child link="ldlidar_base"/>
         <origin xyz="0.122 0 0.212" rpy="0 0 0"/>
     </joint>
-    <link name="laser_frame">
+    <!-- <link name="laser_frame">
         <visual>
             <geometry>
@@ -28,5 +28,22 @@
             <origin xyz="0 0 0" rpy="0 0 0"/>
         </xacro:inertial_cylinder>
+    </link> -->
+    <link name="ldlidar_base">
+        <visual>
+            <origin xyz="0 0 0" rpy="0 0 0"/>
+            <geometry>
+                <mesh filename="package://ldlidar_node/urdf/model/LD19.stl" scale="0.001 0.001 0.001" />
+            </geometry>
+            <material name="ldlidar_mat">
+                <color rgba="0.8 0.8 0.8 0.8"/>
+            </material>
+        </visual>
     </link>
+    <joint name="ldlidar_link_joint" type="fixed">
+        <parent link="ldlidar_base"/>
+        <child link="ldlidar_link"/>
+        <origin xyz="0 0 0.02745" rpy="0 0 0" />
+    </joint>
+    <link name="ldlidar_link" />
     <gazebo reference="laser_frame">
         <material>Gazebo/Black</material>

File: description/ros2_control.xacro (robot description, xacro)
@@ -8,5 +8,5 @@
                 <param name="right_wheel_name">right_wheel_joint</param>
                 <param name="loop_rate">30</param>
-                <param name="device">/dev/ttyUSB0</param>
+                <param name="device">/dev/ttyAMA0</param>
                 <param name="baud_rate">57600</param>
                 <param name="timeout">1000</param>
